File: hardware/can_gps_device/power_supply_3v3_400ma_40V_protected.kicad_sch (KiCad schematic)
At the start: 9 parts, among them U2 TLE42744DV33ATMA1

Commit message: Schematic Initial Rev
Parts:
- renumbered C11 to C10, C12 to C11, C13 to C12
Changed lines of the file:
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@@
 		(dnp no)
 		(fields_autoplaced yes)
-		(property "Reference" "#PWR021"
+		(property "Reference" "#PWR025"
 			(at 153.67 109.22 0)
 			(effects
@@
 			(project "power_supply_3v3_400ma_40V_protected"
 				(path "/742f64ac-c4d8-4561-a2a9-e0e3f6f67ce8/7b74f6f5-1560-4843-a54e-584b3d17c5b1"
-					(reference "#PWR021")
+					(reference "#PWR025")
 					(unit 1)
 				)
@@
 		(dnp no)
 		(fields_autoplaced yes)
-		(property "Reference" "#PWR018"
+		(property "Reference" "#PWR022"
 			(at 115.57 91.44 0)
 			(effects
@@
 			(project ""
 				(path "/742f64ac-c4d8-4561-a2a9-e0e3f6f67ce8/7b74f6f5-1560-4843-a54e-584b3d17c5b1"
-					(reference "#PWR018")
+					(reference "#PWR022")
 					(unit 1)
 				)
@@
 		(on_board yes)
 		(dnp no)
-		(property "Reference" "C12"
+		(property "Reference" "C11"
 			(at 151.13 95.2435 0)
 			(effects
@@
 			(project "power_supply_3v3_400ma_40V_protected"
 				(path "/742f64ac-c4d8-4561-a2a9-e0e3f6f67ce8/7b74f6f5-1560-4843-a54e-584b3d17c5b1"
-					(reference "C12")
+					(reference "C11")
 					(unit 1)
 				)
@@
 		(dnp no)
 		(fields_autoplaced yes)
-		(property "Reference" "#PWR024"
+		(property "Reference" "#PWR028"
 			(at 189.23 92.71 0)
 			(effects
@@
 			(project "power_supply_3v3_400ma_40V_protected"
 				(path "/742f64ac-c4d8-4561-a2a9-e0e3f6f67ce8/7b74f6f5-1560-4843-a54e-584b3d17c5b1"
-					(reference "#PWR024")
+					(reference "#PWR028")
 					(unit 1)
 				)
@@
 		(dnp no)
 		(fields_autoplaced yes)
-		(property "Reference" "#PWR022"
+		(property "Reference" "#PWR026"
 			(at 163.83 109.22 0)
 			(effects
@@
 			(project "power_supply_3v3_400ma_40V_protected"
 				(path "/742f64ac-c4d8-4561-a2a9-e0e3f6f67ce8/7b74f6f5-1560-4843-a54e-584b3d17c5b1"
-					(reference "#PWR022")
+					(reference "#PWR026")
 					(unit 1)
 				)
@@
 		(dnp no)
 		(fields_autoplaced yes)
-		(property "Reference" "#PWR019"
+		(property "Reference" "#PWR023"
 			(at 125.73 116.84 0)
 			(effects
@@
 			(project "power_supply_3v3_400ma_40V_protected"
 				(path "/742f64ac-c4d8-4561-a2a9-e0e3f6f67ce8/7b74f6f5-1560-4843-a54e-584b3d17c5b1"
-					(reference "#PWR019")
+					(reference "#PWR023")
 					(unit 1)
 				)
@@
 		(dnp no)
 		(fields_autoplaced yes)
-		(property "Reference" "#PWR023"
+		(property "Reference" "#PWR027"
 			(at 173.99 107.95 0)
 			(effects
@@
 			(project "power_supply_3v3_400ma_40V_protected"
 				(path "/742f64ac-c4d8-4561-a2a9-e0e3f6f67ce8/7b74f6f5-1560-4843-a54e-584b3d17c5b1"
-					(reference "#PWR023")
+					(reference "#PWR027")
 					(unit 1)
 				)
@@
 		(dnp no)
 		(fields_autoplaced yes)
-		(property "Reference" "#PWR025"
+		(property "Reference" "#PWR029"
 			(at 189.23 116.84 0)
 			(effects
@@
 			(project "power_supply_3v3_400ma_40V_protected"
 				(path "/742f64ac-c4d8-4561-a2a9-e0e3f6f67ce8/7b74f6f5-1560-4843-a54e-584b3d17c5b1"
-					(reference "#PWR025")
+					(reference "#PWR029")
 					(unit 1)
 				)
@@
 		(dnp no)
 		(fields_autoplaced yes)
-		(property "Reference" "C11"
+		(property "Reference" "C10"
 			(at 140.97 95.2435 0)
 			(effects
@@
 			(project "power_supply_3v3_400ma_40V_protected"
 				(path "/742f64ac-c4d8-4561-a2a9-e0e3f6f67ce8/7b74f6f5-1560-4843-a54e-584b3d17c5b1"
-					(reference "C11")
+					(reference "C10")
 					(unit 1)
 				)
@@
 		(dnp no)
 		(fields_autoplaced yes)
-		(property "Reference" "C13"
+		(property "Reference" "C12"
 			(at 176.53 93.9862 0)
 			(effects
@@
 			(project "power_supply_3v3_400ma_40V_protected"
 				(path "/742f64ac-c4d8-4561-a2a9-e0e3f6f67ce8/7b74f6f5-1560-4843-a54e-584b3d17c5b1"
-					(reference "C13")
+					(reference "C12")
 					(unit 1)
 				)
@@
 		(dnp no)
 		(fields_autoplaced yes)
-		(property "Reference" "#PWR020"
+		(property "Reference" "#PWR024"
 			(at 143.51 109.22 0)
 			(effects
@@
 			(project "power_supply_3v3_400ma_40V_protected"
 				(path "/742f64ac-c4d8-4561-a2a9-e0e3f6f67ce8/7b74f6f5-1560-4843-a54e-584b3d17c5b1"
-					(reference "#PWR020")
-					(unit 1)
-				)
+					(reference "#PWR024")
+					(unit 1)
+				)
