File: hardware/can_gps_device/can_transciever_no_term.kicad_sch (KiCad schematic)
At the start: 6 parts, among them U3 TCAN3403DRQ1

Commit message: Schematic Initial Rev
Parts:
- TP1: renamed from TP4; footprint TestPoint:TestPoint_Pad_D1.0mm -> TestPoint:TestPoint_Pad_D1.5mm
- TP2: renamed from TP5; footprint TestPoint:TestPoint_Pad_D1.0mm -> TestPoint:TestPoint_Pad_D1.5mm
- renumbered C14 to C10, C15 to C11, D4 to D3, U3 to U2
Changed lines of the file:
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@@
 		(dnp no)
 		(fields_autoplaced yes)
-		(property "Reference" "TP5"
+		(property "Reference" "TP2"
 			(at 144.78 112.5219 0)
 			(effects
@@
 			)
 		)
-		(property "Footprint" "TestPoint:TestPoint_Pad_D1.0mm"
+		(property "Footprint" "TestPoint:TestPoint_Pad_D1.5mm"
 			(at 137.16 110.49 0)
 			(effects
@@
 			(project "can_transciever_no_term"
 				(path "/742f64ac-c4d8-4561-a2a9-e0e3f6f67ce8/b93d8d5a-c9dc-4552-9959-3cf22fd198ac"
-					(reference "TP5")
+					(reference "TP2")
 					(unit 1)
 				)
@@
 		(dnp no)
 		(fields_autoplaced yes)
-		(property "Reference" "#PWR030"
+		(property "Reference" "#PWR024"
 			(at 162.56 88.9 0)
 			(effects
@@
 			(project "can_transciever_no_term"
 				(path "/742f64ac-c4d8-4561-a2a9-e0e3f6f67ce8/b93d8d5a-c9dc-4552-9959-3cf22fd198ac"
-					(reference "#PWR030")
+					(reference "#PWR024")
 					(unit 1)
 				)
@@
 		(dnp no)
 		(fields_autoplaced yes)
-		(property "Reference" "#PWR028"
+		(property "Reference" "#PWR022"
 			(at 157.48 77.47 0)
 			(effects
@@
 			(project "can_transciever_no_term"
 				(path "/742f64ac-c4d8-4561-a2a9-e0e3f6f67ce8/b93d8d5a-c9dc-4552-9959-3cf22fd198ac"
-					(reference "#PWR028")
+					(reference "#PWR022")
 					(unit 1)
 				)
@@
 		(dnp no)
 		(fields_autoplaced yes)
-		(property "Reference" "#PWR031"
+		(property "Reference" "#PWR025"
 			(at 199.39 101.6 0)
 			(effects
@@
 			(project "can_transciever_no_term"
 				(path "/742f64ac-c4d8-4561-a2a9-e0e3f6f67ce8/b93d8d5a-c9dc-4552-9959-3cf22fd198ac"
-					(reference "#PWR031")
+					(reference "#PWR025")
 					(unit 1)
 				)
@@
 		(on_board yes)
 		(dnp no)
-		(property "Reference" "U3"
+		(property "Reference" "U2"
 			(at 149.86 91.44 0)
 			(effects
@@
 			(project "can_transciever_no_term"
 				(path "/742f64ac-c4d8-4561-a2a9-e0e3f6f67ce8/b93d8d5a-c9dc-4552-9959-3cf22fd198ac"
-					(reference "U3")
+					(reference "U2")
 					(unit 1)
 				)
@@
 		(dnp no)
 		(fields_autoplaced yes)
-		(property "Reference" "#PWR027"
+		(property "Reference" "#PWR021"
 			(at 144.78 85.09 0)
 			(effects
@@
 			(project "can_transciever_no_term"
 				(path "/742f64ac-c4d8-4561-a2a9-e0e3f6f67ce8/b93d8d5a-c9dc-4552-9959-3cf22fd198ac"
-					(reference "#PWR027")
+					(reference "#PWR021")
 					(unit 1)
 				)
@@
 		(dnp no)
 		(fields_autoplaced yes)
-		(property "Reference" "C14"
+		(property "Reference" "C10"
 			(at 138.43 85.0962 0)
 			(effects
@@
 			(project "can_transciever_no_term"
 				(path "/742f64ac-c4d8-4561-a2a9-e0e3f6f67ce8/b93d8d5a-c9dc-4552-9959-3cf22fd198ac"
-					(reference "C14")
+					(reference "C10")
 					(unit 1)
 				)
@@
 		(dnp no)
 		(fields_autoplaced yes)
-		(property "Reference" "#PWR029"
+		(property "Reference" "#PWR023"
 			(at 157.48 121.92 0)
 			(effects
@@
 			(project "can_transciever_no_term"
 				(path "/742f64ac-c4d8-4561-a2a9-e0e3f6f67ce8/b93d8d5a-c9dc-4552-9959-3cf22fd198ac"
-					(reference "#PWR029")
+					(reference "#PWR023")
 					(unit 1)
 				)
@@
 		(dnp no)
 		(fields_autoplaced yes)
-		(property "Reference" "#PWR026"
+		(property "Reference" "#PWR020"
 			(at 135.89 96.52 0)
 			(effects
@@
 			(project "can_transciever_no_term"
 				(path "/742f64ac-c4d8-4561-a2a9-e0e3f6f67ce8/b93d8d5a-c9dc-4552-9959-3cf22fd198ac"
-					(reference "#PWR026")
+					(reference "#PWR020")
 					(unit 1)
 				)
@@
 		(dnp no)
 		(fields_autoplaced yes)
-		(property "Reference" "C15"
+		(property "Reference" "C11"
 			(at 165.1 77.4762 0)
 			(effects
@@
 			(project "can_transciever_no_term"
 				(path "/742f64ac-c4d8-4561-a2a9-e0e3f6f67ce8/b93d8d5a-c9dc-4552-9959-3cf22fd198ac"
-					(reference "C15")
+					(reference "C11")
 					(unit 1)
 				)
@@
 		(on_board yes)
 		(dnp no)
-		(property "Reference" "D4"
+		(property "Reference" "D3"
 			(at 187.198 89.154 90)
 			(effects
@@
 			(project "can_transciever_no_term"
 				(path "/742f64ac-c4d8-4561-a2a9-e0e3f6f67ce8/b93d8d5a-c9dc-4552-9959-3cf22fd198ac"
-					(reference "D4")
+					(reference "D3")
 					(unit 1)
 				)
@@
 		(dnp no)
 		(fields_autoplaced yes)
-		(property "Reference" "TP4"
+		(property "Reference" "TP1"
 			(at 133.35 112.5219 0)
 			(effects
@@
 			)
 		)
-		(property "Footprint" "TestPoint:TestPoint_Pad_D1.0mm"
+		(property "Footprint" "TestPoint:TestPoint_Pad_D1.5mm"
 			(at 125.73 110.49 0)
 			(effects
@@
 			(project "can_transciever_no_term"
 				(path "/742f64ac-c4d8-4561-a2a9-e0e3f6f67ce8/b93d8d5a-c9dc-4552-9959-3cf22fd198ac"
-					(reference "TP4")
-					(unit 1)
-				)
+					(reference "TP1")
+					(unit 1)
+				)

Commit message: PCB design rev 1
Connections:
- net +3V3 renamed +3.3V
Changed lines of the file:
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@@
-	)
-	(symbol
-		(lib_id "power:+3.3V")
-		(at 157.48 73.66 0)
-		(unit 1)
-		(exclude_from_sim no)
-		(in_bom yes)
-		(on_board yes)
-		(dnp no)
-		(fields_autoplaced yes)
-		(property "Reference" "#PWR022"
-			(at 157.48 77.47 0)
-			(effects
-				(font
-					(size 1.27 1.27)
-				)
-				(hide yes)
-			)
-		)
-		(property "Value" "+3V3"
-			(at 157.48 68.58 0)
-			(effects
-				(font
-					(size 1.27 1.27)
-				)
-			)
-		)
-		(property "Footprint" ""
-			(at 157.48 73.66 0)
-			(effects
-				(font
-					(size 1.27 1.27)
-				)
-				(hide yes)
-			)
-		)
-		(property "Datasheet" ""
-			(at 157.48 73.66 0)
-			(effects
-				(font
-					(size 1.27 1.27)
-				)
-				(hide yes)
-			)
-		)
-		(property "Description" ""
-			(at 157.48 73.66 0)
-			(effects
-				(font
-					(size 1.27 1.27)
-				)
-			)
-		)
-		(pin "1"
-		)
-		(instances
-			(project "can_transciever_no_term"
-				(path "/7106a0b2-f612-48d7-957a-fac2f88be8f8"
-					(reference "#PWR?")
-					(unit 1)
-				)
-			)
-			(project "can_transciever_no_term"
-				(path "/742f64ac-c4d8-4561-a2a9-e0e3f6f67ce8/b93d8d5a-c9dc-4552-9959-3cf22fd198ac"
-					(reference "#PWR022")
-					(unit 1)
-				)
-			)
-			(project "canbus_tire_temp_sensor"
-				(path "/e63e39d7-6ac0-4ffd-8aa3-1841a4541b55/5309e4c3-f3b7-4930-9c5f-4b2eb6027320"
-					(reference "#PWR038")
-					(unit 1)
-				)
-			)
-		)
 	)
 	(symbol
@@
 	)
 	(symbol
-		(lib_name "+3.3V_1")
-		(lib_id "power:+3.3V")
-		(at 144.78 81.28 0)
-		(unit 1)
-		(exclude_from_sim no)
-		(in_bom yes)
-		(on_board yes)
-		(dnp no)
-		(fields_autoplaced yes)
-		(property "Reference" "#PWR021"
-			(at 144.78 85.09 0)
-			(effects
-				(font
-					(size 1.27 1.27)
-				)
-				(hide yes)
-			)
-		)
-		(property "Value" "+3V3"
-			(at 144.78 76.2 0)
-			(effects
-				(font
-					(size 1.27 1.27)
-				)
-			)
-		)
-		(property "Footprint" ""
-			(at 144.78 81.28 0)
-			(effects
-				(font
-					(size 1.27 1.27)
-				)
-				(hide yes)
-			)
-		)
-		(property "Datasheet" ""
-			(at 144.78 81.28 0)
-			(effects
-				(font
-					(size 1.27 1.27)
-				)
-				(hide yes)
-			)
-		)
-		(property "Description" ""
-			(at 144.78 81.28 0)
-			(effects
-				(font
-					(size 1.27 1.27)
-				)
-			)
-		)
-		(pin "1"
-		)
-		(instances
-			(project "can_transciever_no_term"
-				(path "/7106a0b2-f612-48d7-957a-fac2f88be8f8"
-					(reference "#PWR?")
-					(unit 1)
-				)
-			)
-			(project "can_transciever_no_term"
-				(path "/742f64ac-c4d8-4561-a2a9-e0e3f6f67ce8/b93d8d5a-c9dc-4552-9959-3cf22fd198ac"
-					(reference "#PWR021")
-					(unit 1)
-				)
-			)
-			(project "canbus_tire_temp_sensor"
-				(path "/e63e39d7-6ac0-4ffd-8aa3-1841a4541b55/5309e4c3-f3b7-4930-9c5f-4b2eb6027320"
-					(reference "#PWR037")
-					(unit 1)
-				)
-			)
-		)
-	)
-	(symbol
 		(lib_id "Device:C_Small")
 		(at 135.89 86.36 0)
@@
 	)
 	(symbol
+		(lib_name "+3.3V_2")
+		(lib_id "power:+3.3V")
+		(at 144.78 81.28 0)
+		(unit 1)
+		(exclude_from_sim no)
+		(in_bom yes)
+		(on_board yes)
+		(dnp no)
+		(fields_autoplaced yes)
+		(property "Reference" "#PWR050"
+			(at 144.78 85.09 0)
+			(effects
+				(font
+					(size 1.27 1.27)
+				)
+				(hide yes)
+			)
+		)
+		(property "Value" "+3.3V"
+			(at 144.78 76.2 0)
+			(effects
+				(font
+					(size 1.27 1.27)
+				)
+			)
+		)
+		(property "Footprint" ""
+			(at 144.78 81.28 0)
+			(effects
+				(font
+					(size 1.27 1.27)
+				)
+				(hide yes)
+			)
+		)
+		(property "Datasheet" ""
+			(at 144.78 81.28 0)
+			(effects
+				(font
+					(size 1.27 1.27)
+				)
+				(hide yes)
+			)
+		)
+		(property "Description" "Power symbol creates a global label with name \"+3.3V\""
+			(at 144.78 81.28 0)
+			(effects
+				(font
+					(size 1.27 1.27)
+				)
+				(hide yes)
+			)
+		)
+		(pin "1"
+		)
+		(instances
+			(project "can_gps_device"
+				(path "/742f64ac-c4d8-4561-a2a9-e0e3f6f67ce8/b93d8d5a-c9dc-4552-9959-3cf22fd198ac"
+					(reference "#PWR050")
+					(unit 1)
+				)
+			)
+		)
+	)
+	(symbol
 		(lib_id "Device:C_Small")
 		(at 162.56 78.74 0)
@@
 					(unit 1)
 				)
+			)
+		)
+	)
+	(symbol
+		(lib_name "+3.3V_2")
+		(lib_id "power:+3.3V")
+		(at 157.48 73.66 0)
+		(unit 1)
+		(exclude_from_sim no)
+		(in_bom yes)
+		(on_board yes)
+		(dnp no)
+		(fields_autoplaced yes)
+		(property "Reference" "#PWR047"
+			(at 157.48 77.47 0)
+			(effects
+				(font
+					(size 1.27 1.27)
+				)
+				(hide yes)
+			)
+		)
+		(property "Value" "+3.3V"
+			(at 157.48 68.58 0)
+			(effects
+				(font
+					(size 1.27 1.27)
+				)
+			)
+		)
+		(property "Footprint" ""
+			(at 157.48 73.66 0)
+			(effects
+				(font
+					(size 1.27 1.27)
+				)
+				(hide yes)
+			)
+		)
+		(property "Datasheet" ""
+			(at 157.48 73.66 0)
+			(effects
+				(font
+					(size 1.27 1.27)
+				)
+				(hide yes)
+			)
+		)
+		(property "Description" "Power symbol creates a global label with name \"+3.3V\""
+			(at 157.48 73.66 0)
+			(effects
+				(font
+					(size 1.27 1.27)
+				)
+				(hide yes)
+			)
+		)
+		(pin "1"
+		)
+		(instances
+			(project ""
+				(path "/742f64ac-c4d8-4561-a2a9-e0e3f6f67ce8/b93d8d5a-c9dc-4552-9959-3cf22fd198ac"
+					(reference "#PWR047")
+					(unit 1)
+				)
