File: hardware/can_gps_device/gps_ublox_max-f10s.kicad_sch (KiCad schematic)
At the start: 1 part

Commit message: Schematic Initial Rev
Parts:
- removed U4: ~, symbol RF_GPS:MAX-F10S
- added C12: 1uF, Capacitor_SMD:C_0603_1608Metric, symbol Device:C_Small
- added C13: 0.1uF, Capacitor_SMD:C_0603_1608Metric, symbol Device:C_Small
- added C14: 100nF 16V X7R, Capacitor_SMD:C_0603_1608Metric, symbol Device:C_Small
- added C15: FYD0H104ZF, Capacitor_THT:CP_Radial_D13.0mm_P5.00mm, symbol Device:C_Polarized
- added D4: BAT54A, Package_TO_SOT_SMD:SOT-23, symbol Diode:BAT54A
- added D5: ESD9R3.3ST5G, Diode_SMD:D_SOD-923, symbol Device:D_TVS
- added J3: SMA-J-P-X-RA-TH1, can_gps_device:SAMTEC_SMA-J-P-X-RA-TH1, symbol can_gps_device:SMA-J-P-X-RA-TH1
- added JP2: Jumper_2_Bridged, Jumper:SolderJumper-2_P1.3mm_Bridged_RoundedPad1.0x1.5mm, symbol Jumper:Jumper_2_Bridged
- added L1: LQG15HN27NJ02D, Inductor_SMD:L_0402_1005Metric_Pad0.77x0.64mm_HandSolder, symbol Device:L
- added MCU_RX1, MCU_TX1: TestPoint, TestPoint:TestPoint_Pad_D1.5mm, symbol Connector:TestPoint
- added R5: 22 1/2 W 1206, Resistor_SMD:R_1206_3216Metric, symbol Device:R_Small
- added R6: 470, Resistor_SMD:R_0603_1608Metric, symbol Device:R_Small
- added U3: NEO-M9V-20B, can_gps_device:XCVR_NEO-M9V-20B, symbol can_gps_device:NEO-M9V-20B
Connections:
- net +3V3: now also C12.1, U3.2 (D_SEL), U3.23 (VCC)
- net GND: now also C12.2, C13.2, C14.2, C15.2, D5.1 (A1), J3.2, J3.3, J3.4, J3.5, U3.10 (GND), U3.12 (GND__1), U3.13 (GND__2), U3.14 (LNA_EN), U3.24 (GND__3), U3.7 (V_USB)
- net GNSS_RESET: now also U3.8 (~{RESET})
- net RF_IN: now also D5.2 (A2), J3.1, L1.1, U3.11 (RF_IN)
- net VCC_RF: now also R5.2, U3.9 (VCC_RF)
- new net: C14.1, L1.2, R5.1
- new net: D4.2, R6.1
- new net: C13.1, JP2.1 (A), U3.22 (V_BCKP)
- new net +3.3V: D4.3
- new net +BATT_BCKP: C15.1, JP2.2 (B), R6.2
- new net GNSS_TIMEPULSE: U3.3 (TIMEPULSE)
- new net GNSS_WAKE_ON_MOTION: U3.17 (WOM)
- new net UART_MCU_RX: MCU_RX1.1, U3.20 (TXD/SPI_MISO)
- new net UART_MCU_TX: MCU_TX1.1, U3.21 (RXD/SPI_MOSI)
- no-connect marks 6 -> 9
Other:
- note added: "100 mF 5.5V"
- note added: "ANN-MB5 has SMA (plug) connector"
- note added: "Backup operating voltage: 1.65 - 3.6 V Backup current: 45 uA typical Target backup operating time: 30 min (1800 s)"
- note added: "Charge path: - diode prevents backfeed - current limiting resistor for inrush"
- note added: "Expected supercap lifetime: LS = Lr * 2X * 2Y X = (Tm-Ta)/10 Y = (Vr-Va)/0.2 LS = 2000 * 2*(70 - 50)/10 *(5.5-3.3)/0.2 LS = 88,000 hours"
- note added: "GNSS + IMU Dead Reckoning Module"
- note added: "I = Q / t C = Q1 / V_low C = Q2 / V_high Q = Q2 - Q1 t = (Q2 - Q1) / I t = C * (V_high - V_low) / I C = t * I / (V_high_V_low) 1.5 safety factor (1800 * 1.5) * 45E-6 / (3.3 - 0.2 - 1.65) = 84 mF minimum"
- note added: "Keep digital return currents away from RF ground."
- note added: "LNA_EN -> external LNA disabled"
- note added: "Layout notes: - RF_IN must have 50 ohm characteristic impedance - use GND via wall around microstrip - no stubs"
- note added: "Limits short circuit current to 150 mA"
- note added: "RF Circuit"
- note added: "Supercap backup supply"
- note added: "~0.2V drop @ 5mA"
- note removed: "Default Interface: - UART 9600 baudrate - 8 bit no parit, 1 stop"
- note removed: "Power consumption: 100 mA max inrush, ~25 mA @ 3.3V supply"
- note removed: "RF_IN: 50 ohm characteristic impedance on transmission line"

Commit message: PCB design rev 1
Connections:
- net +3V3 is gone; now on net +3.3V: C12.1, U3.2 (D_SEL), U3.23 (VCC)
Changed lines of the file:
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@@
+	)
+	(symbol
+		(lib_id "power:+3.3V")
+		(at 100.33 88.9 0)
+		(unit 1)
+		(exclude_from_sim no)
+		(in_bom yes)
+		(on_board yes)
+		(dnp no)
+		(fields_autoplaced yes)
+		(property "Reference" "#PWR021"
+			(at 100.33 92.71 0)
+			(effects
+				(font
+					(size 1.27 1.27)
+				)
+				(hide yes)
+			)
+		)
+		(property "Value" "+3.3V"
+			(at 100.33 83.82 0)
+			(effects
+				(font
+					(size 1.27 1.27)
+				)
+			)
+		)
+		(property "Footprint" ""
+			(at 100.33 88.9 0)
+			(effects
+				(font
+					(size 1.27 1.27)
+				)
+				(hide yes)
+			)
+		)
+		(property "Datasheet" ""
+			(at 100.33 88.9 0)
+			(effects
+				(font
+					(size 1.27 1.27)
+				)
+				(hide yes)
+			)
+		)
+		(property "Description" "Power symbol creates a global label with name \"+3.3V\""
+			(at 100.33 88.9 0)
+			(effects
+				(font
+					(size 1.27 1.27)
+				)
+				(hide yes)
+			)
+		)
+		(pin "1"
+		)
+		(instances
+			(project ""
+				(path "/742f64ac-c4d8-4561-a2a9-e0e3f6f67ce8/43a9972b-cf0d-4376-a58f-5e3d25a0f170"
+					(reference "#PWR021")
+					(unit 1)
+				)
+			)
+		)
 	)
 	(symbol
@@
 	)
 	(symbol
-		(lib_id "power:+3V3")
+		(lib_id "power:GND")
+		(at 228.6 69.85 0)
+		(unit 1)
+		(exclude_from_sim no)
+		(in_bom yes)
+		(on_board yes)
+		(dnp no)
+		(fields_autoplaced yes)
+		(property "Reference" "#PWR037"
+			(at 228.6 76.2 0)
+			(effects
+				(font
+					(size 1.27 1.27)
+				)
+				(hide yes)
+			)
+		)
+		(property "Value" "RF_GND"
+			(at 228.6 74.93 0)
+			(effects
+				(font
+					(size 1.27 1.27)
+				)
+			)
+		)
+		(property "Footprint" ""
+			(at 228.6 69.85 0)
+			(effects
+				(font
+					(size 1.27 1.27)
+				)
+				(hide yes)
+			)
+		)
+		(property "Datasheet" ""
+			(at 228.6 69.85 0)
+			(effects
+				(font
+					(size 1.27 1.27)
+				)
+				(hide yes)
+			)
+		)
+		(property "Description" "Power symbol creates a global label with name \"GND\" , ground"
+			(at 228.6 69.85 0)
+			(effects
+				(font
+					(size 1.27 1.27)
+				)
+				(hide yes)
+			)
+		)
+		(pin "1"
+		)
+		(instances
+			(project "can_gps_device"
+				(path "/742f64ac-c4d8-4561-a2a9-e0e3f6f67ce8/43a9972b-cf0d-4376-a58f-5e3d25a0f170"
+					(reference "#PWR037")
+					(unit 1)
+				)
+			)
+		)
+	)
+	(symbol
+		(lib_id "power:+3.3V")
 		(at 49.53 137.16 90)
 		(unit 1)
@@
 		(on_board yes)
 		(dnp no)
-		(property "Reference" "#PWR026"
+		(fields_autoplaced yes)
+		(property "Reference" "#PWR022"
 			(at 53.34 137.16 0)
 			(effects
@@
 			)
 		)
-		(property "Value" "+3V3"
-			(at 43.942 137.16 90)
-			(effects
-				(font
-					(size 1.27 1.27)
-				)
+		(property "Value" "+3.3V"
+			(at 45.72 137.1599 90)
+			(effects
+				(font
+					(size 1.27 1.27)
+				)
+				(justify left)
 			)
 		)
@@
 			)
 		)
-		(property "Description" "Power symbol creates a global label with name \"+3V3\""
+		(property "Description" "Power symbol creates a global label with name \"+3.3V\""
 			(at 49.53 137.16 0)
 			(effects
@@
 			(project "can_gps_device"
 				(path "/742f64ac-c4d8-4561-a2a9-e0e3f6f67ce8/43a9972b-cf0d-4376-a58f-5e3d25a0f170"
-					(reference "#PWR026")
-					(unit 1)
-				)
-			)
-		)
-	)
-	(symbol
-		(lib_id "power:GND")
-		(at 228.6 69.85 0)
-		(unit 1)
-		(exclude_from_sim no)
-		(in_bom yes)
-		(on_board yes)
-		(dnp no)
-		(fields_autoplaced yes)
-		(property "Reference" "#PWR037"
-			(at 228.6 76.2 0)
-			(effects
-				(font
-					(size 1.27 1.27)
-				)
-				(hide yes)
-			)
-		)
-		(property "Value" "RF_GND"
-			(at 228.6 74.93 0)
-			(effects
-				(font
-					(size 1.27 1.27)
-				)
-			)
-		)
-		(property "Footprint" ""
-			(at 228.6 69.85 0)
-			(effects
-				(font
-					(size 1.27 1.27)
-				)
-				(hide yes)
-			)
-		)
-		(property "Datasheet" ""
-			(at 228.6 69.85 0)
-			(effects
-				(font
-					(size 1.27 1.27)
-				)
-				(hide yes)
-			)
-		)
-		(property "Description" "Power symbol creates a global label with name \"GND\" , ground"
-			(at 228.6 69.85 0)
-			(effects
-				(font
-					(size 1.27 1.27)
-				)
-				(hide yes)
-			)
-		)
-		(pin "1"
-		)
-		(instances
-			(project "can_gps_device"
-				(path "/742f64ac-c4d8-4561-a2a9-e0e3f6f67ce8/43a9972b-cf0d-4376-a58f-5e3d25a0f170"
-					(reference "#PWR037")
+					(reference "#PWR022")
 					(unit 1)
 				)
@@
 					(unit 1)
 				)
-			)
-		)
-	)
-	(symbol
-		(lib_id "power:+3V3")
-		(at 100.33 88.9 0)
-		(unit 1)
-		(exclude_from_sim no)
-		(in_bom yes)
-		(on_board yes)
-		(dnp no)
-		(fields_autoplaced yes)
-		(property "Reference" "#PWR028"
-			(at 100.33 92.71 0)
-			(effects
-				(font
-					(size 1.27 1.27)
-				)
-				(hide yes)
-			)
-		)
-		(property "Value" "+3V3"
-			(at 100.33 83.82 0)
-			(effects
-				(font
-					(size 1.27 1.27)
-				)
-			)
-		)
-		(property "Footprint" ""
-			(at 100.33 88.9 0)
-			(effects
-				(font
-					(size 1.27 1.27)
-				)
-				(hide yes)
-			)
-		)
-		(property "Datasheet" ""
-			(at 100.33 88.9 0)
-			(effects
-				(font
-					(size 1.27 1.27)
-				)
-				(hide yes)
-			)
-		)
-		(property "Description" "Power symbol creates a global label with name \"+3V3\""
-			(at 100.33 88.9 0)
-			(effects
-				(font
-					(size 1.27 1.27)
-				)
-				(hide yes)
-			)
-		)
-		(pin "1"
-		)
-		(instances
-			(project ""
-				(path "/742f64ac-c4d8-4561-a2a9-e0e3f6f67ce8/43a9972b-cf0d-4376-a58f-5e3d25a0f170"
-					(reference "#PWR028")
-					(unit 1)
-				)
