File: hardware/can_gps_device/can_gps_device.kicad_sch (KiCad schematic)
At the start: 5 parts, among them J1 AMP_Superseal_9-6437287-8

Commit message: Schematic Initial Rev
Parts:
- removed J1: AMP_Superseal_9-6437287-8, signal_to_can:TE_9-6437287-8_1, symbol signal-to-can:AMP_Superseal_9-6437287-8
- added J1: Conn_01x04, can_gps_device:ATF13-4P-BM13_AMP, symbol Connector_Generic:Conn_01x04
Connections:
- net +BATT: now also J1.1 (Pin_1)
- net CAN_N: now also J1.3 (Pin_3)
- net CAN_P: now also J1.2 (Pin_2)
- net GND: now also J1.4 (Pin_4)
Other:
- removed sheet 3.3V Linear Regulator
- added sheet 3.3V Switching Regulator (power_supply_switching_module_3.3V.kicad_sch)
- sheet GPS Module ports: added GNSS_RESET, GNSS_TIMEPULSE, GNSS_WAKE_ON_MOTION, UART_MCU_RX, UART_MCU_TX; removed none
- sheet Microcontroller ports: added GNSS_RESET, GNSS_TIMEPULSE, GNSS_WAKE_ON_MOTION, UART_MCU_RX, UART_MCU_TX; removed 3.3V_ANALOG_INPUT_0, 3.3V_ANALOG_INPUT_1, 3.3V_ANALOG_INPUT_2, 3.3V_ANALOG_INPUT_3, 3.3V_ANALOG_INPUT_4, 3.3V_ANALOG_INPUT_5, 3.3V_ANALOG_INPUT_6, 3.3V_ANALOG_INPUT_7
- note added: "PCB Header: ATPF13-4P-BM13 - Deutsch DTM, Amphenol ATP compatible - 4 position, right angle Mating Part: DTM06-4P, ATP06-4P"
- note removed: "PCB Header: 9-6437287-8 - 26 pin, 4 row - keying type: 1 - locking type: upper Mating Part: 3-1437290-7 Mating Part terminals: 3-1447221-3 (18-22 awg) Cavity Plug: 4-1437284-3"
- moved on the sheet: H1, H2, H3, H4

Commit message: Updated MX config and schematic PDF
Other:
- note added: "PCB Stackup Requirement: 4 layer JLC04161H-7628"
Changed lines of the file:
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@@
+		)
+	)
+	(text "PCB Stackup Requirement: 4 layer JLC04161H-7628"
+		(exclude_from_sim no)
+		(at 14.732 42.418 0)
+		(effects
+			(font
+				(size 1.27 1.27)
+			)
+			(justify left)
 		)
 	)
@@
 	)
 	(sheet
-		(at 96.52 138.43)
-		(size 50.8 12.7)
+		(at 97.79 124.46)
+		(size 50.8 16.51)
 		(exclude_from_sim no)
 		(in_bom yes)
@@
 		)
 		(property "Sheetname" "3.3V Switching Regulator"
-			(at 96.52 137.7184 0)
+			(at 97.79 123.7484 0)
 			(effects
 				(font
@@
 		)
 		(property "Sheetfile" "power_supply_switching_module_3.3V.kicad_sch"
-			(at 96.52 151.7146 0)
-			(effects
-				(font
+			(at 97.79 141.5546 0)
+			(effects
+				(font
