File: hardware/can_gps_device/stm32f042k6ux.kicad_sch (KiCad schematic)
At the start: 20 parts, among them J2 TC2030, U1 STM32F042K6Ux, Y1 ECS-160-10-36Q-AES-TR

Commit message: Schematic Initial Rev
Parts:
- removed C4: 0.1uF, Capacitor_SMD:C_0603_1608Metric, symbol Device:C_Small
- added RESET1: TestPoint, TestPoint:TestPoint_Pad_D1.5mm, symbol Connector:TestPoint
- C3: renamed from C2; value 4.7uF -> 0.1uF
- C4: renamed from C5; value 0.1uF -> 4.7uF
- D1, D2: value LED -> Green LED
- renumbered C3 to C2, C6 to C5, C7 to C6, C8 to C7, C9 to C8, C10 to C9
Connections:
- net CAN_STANDBY: now also U1.25 (PA15); no longer U1.27 (PB4)
- net LED_STATUS_1: now also U1.27 (PB4); no longer U1.14 (PB0)
- net LED_STATUS_2: now also U1.26 (PB3); no longer U1.15 (PB1)
- net NRST: now also RESET1.1
- net GNSS_WAKE_ON_MOTION: now reaches U1.16 (PB2)
- net UART_MCU_TX: now reaches U1.19 (PA9)
- net UART_MCU_RX: now reaches U1.20 (PA10)
- net +3V3 renamed +3.3V
- net 3.3V_ANALOG_INPUT_0: no longer names the net of U1.6 (PA0)
- net 3.3V_ANALOG_INPUT_1: no longer names the net of U1.7 (PA1)
- net 3.3V_ANALOG_INPUT_2: no longer names the net of U1.8 (PA2)
- net 3.3V_ANALOG_INPUT_3: no longer names the net of U1.9 (PA3)
- net 3.3V_ANALOG_INPUT_4: no longer names the net of U1.10 (PA4)
- net 3.3V_ANALOG_INPUT_5: no longer names the net of U1.11 (PA5)
- net 3.3V_ANALOG_INPUT_6: no longer names the net of U1.12 (PA6)
- net 3.3V_ANALOG_INPUT_7: no longer names the net of U1.13 (PA7)
- new net GNSS_RESET: U1.15 (PB1)
- new net GNSS_TIMEPULSE: U1.14 (PB0)
- no-connect marks 11 -> 14
Other:
- note added: "16 Mhz HSE"
- note added: "BOOT0 -> 3.3V: Boot to system memory BOOT0 -> GND: Boot to flash memory (normal"
- note added: "CubeMX Setup"
- note added: "Note: no reset button"
- note added: "Status LEDs"
- note added: "TC2030-NL Programming"
- note added: "VDD Pin"
- note added: "VDDA Pin"
- note added: "VDDIO2 Pin"
- moved on the sheet: C1, C2, C3, C4, C5, C6, C7, C8, C9, D1, D2, J2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

Commit message: PCB design rev 1
Connections:
- net GNSS_RESET: now also U1.14 (PB0); no longer U1.15 (PB1)
- net GNSS_TIMEPULSE: now also U1.16 (PB2); no longer U1.14 (PB0)
- net GNSS_WAKE_ON_MOTION: now also U1.15 (PB1); no longer U1.16 (PB2)
Changed lines of the file:
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@@
 	(wire
 		(pts
-			(xy 213.36 54.61) (xy 215.9 54.61)
+			(xy 35.56 135.89) (xy 67.31 135.89)
 		)
 		(stroke
@@
 	(wire
 		(pts
-			(xy 35.56 135.89) (xy 67.31 135.89)
+			(xy 116.84 77.47) (xy 119.38 77.47)
 		)
 		(stroke
@@
 	(wire
 		(pts
-			(xy 116.84 77.47) (xy 119.38 77.47)
+			(xy 213.36 54.61) (xy 215.9 54.61)
 		)
 		(stroke
@@
 	(wire
 		(pts
-			(xy 213.36 59.69) (xy 215.9 59.69)
-		)
-		(stroke
-			(width 0)
-			(type default)
-		)
-	)
-	(wire
-		(pts
 			(xy 119.38 77.47) (xy 121.92 77.47)
 		)
@@
 	(wire
 		(pts
-			(xy 213.36 57.15) (xy 215.9 57.15)
-		)
-		(stroke
-			(width 0)
-			(type default)
-		)
-	)
-	(wire
-		(pts
 			(xy 129.54 85.09) (xy 129.54 86.36)
 		)
@@
 	(wire
 		(pts
+			(xy 213.36 57.15) (xy 215.9 57.15)
+		)
+		(stroke
+			(width 0)
+			(type default)
+		)
+	)
+	(wire
+		(pts
 			(xy 74.93 72.39) (xy 74.93 74.93)
 		)
@@
 	(wire
 		(pts
+			(xy 213.36 59.69) (xy 215.9 59.69)
+		)
+		(stroke
+			(width 0)
+			(type default)
+		)
+	)
+	(wire
+		(pts
 			(xy 74.93 82.55) (xy 74.93 85.09)
 		)
@@
 	(hierarchical_label "GNSS_TIMEPULSE"
 		(shape input)
-		(at 213.36 54.61 180)
+		(at 213.36 59.69 180)
 		(effects
 			(font
@@
 	(hierarchical_label "GNSS_RESET"
 		(shape output)
-		(at 213.36 57.15 180)
+		(at 213.36 54.61 180)
 		(effects
 			(font
@@
 	(hierarchical_label "GNSS_WAKE_ON_MOTION"
 		(shape input)
-		(at 213.36 59.69 180)
+		(at 213.36 57.15 180)
 		(effects
 			(font

Commit message: Updated MX config and schematic PDF
Other:
- note added: "BOOT0 -> 3.3V: Boot to system memory BOOT0 -> GND: Boot to flash memory (normal)"
- note removed: "BOOT0 -> 3.3V: Boot to system memory BOOT0 -> GND: Boot to flash memory (normal"
